File: PCB/constellation.kicad_pcb (KiCad board)
At the start: 2 copper layers, 104.8 x 104.8 mm, 23 parts, among them SW1 SW_SPST

Commit message: silkscreen
Other:
- board text added: "CONSTELLATION"
- board text added: "SAGITTARIUS"
- board text added: "made with love and patience - rudransh goel"
